File: amiga-500-usb-kb-RP2040 (rev0)/amiga-500-usb-kb-rp2040.kicad_pcb (KiCad board)
At the start: 4 copper layers, 42.5 x 40 mm, 44 parts, among them IC1 TXS0104ED, IC2 W25Q64JVXGIQ_TR, IC3 TPS7A2033PDBVR, J1 47346-0001, J2 USB_HEADER, J3 Type A, J4 Type B, J5 Power LED, J6 Floppy LED, U0 RP2040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

Commit message: Add files via upload
Other:
- board text added: "wiretap 2024"
